Commit message: nav2 stuff

File: description/robot_core_2.xacro (robot description, xacro)
@@ -30,4 +30,10 @@
     <!-- BASE LINK-->
     <link name="base_link"></link>
+    <joint name="base_footprint_joint" type="fixed">
+        <parent link="base_link"/>
+        <child link="base_footprint"/>
+        <origin xyz="0 0 0" rpy="0 0 0"/>
+    </joint>
+    <link name="base_footprint"></link>
     <!-- CHASSIS-->
     <joint name="chassis_joint" type="fixed">
