Commit message: edited urdf and meshes

File: description/robot.urdf.xacro (robot description, xacro)
@@ -6,17 +6,17 @@
         <origin xyz="0 0 0" rpy="0 0 0"/>
         <mass value="1.0"/>
-        <inertia ixx="288.5336" ixy="0" ixz="-1e-05" iyy="274.41498" iyz="0" izz="149.48827"/>
+        <inertia ixx="288.5336" ixy="0" ixz="0" iyy="274.41498" iyz="0" izz="149.48827"/>
       </inertial>
       <visual name="camera">
-        <origin xyz="0 0 0" rpy="0 -1.5708 0"/>
+        <origin xyz="0 0 0" rpy="0 0 0"/>
         <geometry>
-          <mesh filename="..\meshes\dae\Cube.018.dae" scale="1.0 1.0 1.0"/>
+          <mesh filename="file://$(find wally)/meshes/dae/Cube.018.dae" scale="1.0 1.0 1.0"/>
         </geometry>
         <material name="black"/>
       </visual>
       <collision name="camera">
-        <origin xyz="-0.05651 -0.0476 0.12457" rpy="0 -1.5708 0"/>
+        <origin xyz="0.00012 -5e-05 6e-05" rpy="0 0 0"/>
         <geometry>
-          <mesh filename="..\meshes\dae\Cube.028.dae" scale="1.0 1.0 1.0"/>
+          <mesh filename="file://$(find wally)/meshes/dae/Cube.028.dae" scale="1.0 1.0 1.0"/>
         </geometry>
       </collision>
@@ -26,17 +26,17 @@
         <origin xyz="0 0 0" rpy="0 0 0"/>
         <mass value="1.0"/>
-        <inertia ixx="2658.80078" ixy="-0.00068" ixz="0" iyy="4901.40967" iyz="0" izz="5801.34521"/>
+        <inertia ixx="2658.80078" ixy="0" ixz="0" iyy="4901.40967" iyz="0" izz="5801.34521"/>
       </inertial>
       <visual name="chassis">
-        <origin xyz="0 0 0" rpy="0 0 3.14159"/>
+        <origin xyz="0 0 0" rpy="0 0 0"/>
         <geometry>
-          <mesh filename="..\meshes\dae\Cube.023.dae" scale="1.0 1.0 1.0"/>
+          <mesh filename="file://$(find wally)/meshes/dae/Cube.023.dae" scale="1.0 1.0 1.0"/>
         </geometry>
         <material name="yellow"/>
       </visual>
       <collision name="chassis">
-        <origin xyz="-0.08775 -0.613 0.10621" rpy="0 0 3.14159"/>
+        <origin xyz="9e-05 0.00061 0.00011" rpy="0 0 0"/>
         <geometry>
-          <mesh filename="..\meshes\dae\Cube.026.dae" scale="1.0 1.0 1.0"/>
+          <mesh filename="file://$(find wally)/meshes/dae/Cube.026.dae" scale="1.0 1.0 1.0"/>
         </geometry>
       </collision>
@@ -51,12 +51,12 @@
         <origin xyz="0 0 0" rpy="0 0 0"/>
         <geometry>
-          <mesh filename="..\meshes\dae\Cube.019.dae" scale="1.0 1.0 1.0"/>
+          <mesh filename="file://$(find wally)/meshes/dae/Cube.019.dae" scale="1.0 1.0 1.0"/>
         </geometry>
         <material name="black"/>
       </visual>
       <collision name="laser">
-        <origin xyz="0 0 -0.02138" rpy="0 0 0"/>
+        <origin xyz="0 0 -2e-05" rpy="0 0 0"/>
         <geometry>
-          <mesh filename="..\meshes\dae\Cube.027.dae" scale="1.0 1.0 1.0"/>
+          <mesh filename="file://$(find wally)/meshes/dae/Cube.027.dae" scale="1.0 1.0 1.0"/>
         </geometry>
       </collision>
@@ -71,5 +71,5 @@
         <origin xyz="0 0 0" rpy="0 0 0"/>
         <geometry>
-          <mesh filename="..\meshes\dae\Cube.020.dae" scale="1.0 1.0 1.0"/>
+          <mesh filename="file://$(find wally)/meshes/dae/Cube.020.dae" scale="1.0 1.0 1.0"/>
         </geometry>
         <material name="black"/>
@@ -80,17 +80,17 @@
         <origin xyz="0 0 0" rpy="0 0 0"/>
         <mass value="1.0"/>
-        <inertia ixx="289.20636" ixy="0" ixz="0" iyy="506.04105" iyz="-2e-05" izz="289.19714"/>
+        <inertia ixx="289.20636" ixy="0" ixz="0" iyy="506.04105" iyz="0" izz="289.19714"/>
       </inertial>
       <visual name="wheel_left">
-        <origin xyz="0 0 0" rpy="1.5708 0 0"/>
+        <origin xyz="0 0 0" rpy="0 0 0"/>
         <geometry>
-          <mesh filename="..\meshes\dae\Cube.022.dae" scale="1.0 1.0 1.0"/>
+          <mesh filename="file://$(find wally)/meshes/dae/Cube.022.dae" scale="1.0 1.0 1.0"/>
         </geometry>
         <material name="yellow"/>
       </visual>
       <collision name="wheel_left">
-        <origin xyz="0.01732 -0.02453 -0.10548" rpy="1.5708 0 0"/>
+        <origin xyz="2e-05 -0.00011 2e-05" rpy="0 0 0"/>
         <geometry>
-          <mesh filename="..\meshes\dae\Cube.025.dae" scale="1.0 1.0 1.0"/>
+          <mesh filename="file://$(find wally)/meshes/dae/Cube.025.dae" scale="1.0 1.0 1.0"/>
         </geometry>
       </collision>
@@ -100,47 +100,47 @@
         <origin xyz="0 0 0" rpy="0 0 0"/>
         <mass value="1.0"/>
-        <inertia ixx="289.20636" ixy="0" ixz="0" iyy="506.04105" iyz="2e-05" izz="289.19717"/>
+        <inertia ixx="289.20636" ixy="0" ixz="0" iyy="506.04105" iyz="0" izz="289.19717"/>
       </inertial>
       <visual name="wheel_right">
-        <origin xyz="0 0 0" rpy="-1.5708 0 0"/>
+        <origin xyz="0 0 0" rpy="0 0 0"/>
         <geometry>
-          <mesh filename="..\meshes\dae\Cube.017.dae" scale="1.0 1.0 1.0"/>
+          <mesh filename="file://$(find wally)/meshes/dae/Cube.017.dae" scale="1.0 1.0 1.0"/>
         </geometry>
         <material name="yellow"/>
       </visual>
       <collision name="wheel_right">
-        <origin xyz="0.01732 0.02454 -2.55418" rpy="-1.5708 0 0"/>
+        <origin xyz="2e-05 0.00255 2e-05" rpy="0 0 0"/>
         <geometry>
-          <mesh filename="..\meshes\dae\Cube.024.dae" scale="1.0 1.0 1.0"/>
+          <mesh filename="file://$(find wally)/meshes/dae/Cube.024.dae" scale="1.0 1.0 1.0"/>
         </geometry>
       </collision>
     </link>
     <joint name="link_camera" type="fixed">
-      <origin xyz="-99.50021 -0.66059 75.61109" rpy="-3.14159 1.5708 0"/>
+      <origin xyz="0.0995 0.00066 0.07561" rpy="0 0 0"/>
       <parent link="link_chassis"/>
       <child link="link_camera"/>
     </joint>
     <joint name="link_laser" type="fixed">
-      <origin xyz="13.13231 -0.613 104.50001" rpy="0 0 3.14159"/>
+      <origin xyz="-0.01313 0.00061 0.1045" rpy="0 0 0"/>
       <parent link="link_chassis"/>
       <child link="link_laser"/>
     </joint>
     <joint name="link_wheel_caster" type="fixed">
-      <origin xyz="98.95988 -0.61332 -7.88988" rpy="0 0 3.14159"/>
+      <origin xyz="-0.09896 0.00061 -0.00789" rpy="0 0 0"/>
       <parent link="link_chassis"/>
       <child link="link_wheel_caster"/>
     </joint>
     <joint name="link_wheel_left" type="revolute">
-      <origin xyz="-6.02121 -77.0348 16.15401" rpy="-1.5708 0 3.14159"/>
+      <origin xyz="0.00602 0.07703 0.01615" rpy="0 0 0"/>
       <parent link="link_chassis"/>
       <child link="link_wheel_left"/>
-      <axis xyz="0 0 1.0"/>
+      <axis xyz="0 1.0 0"/>
       <limit lower="-3.14" upper="3.14" effort="0" velocity="0"/>
     </joint>
     <joint name="link_wheel_right" type="revolute">
-      <origin xyz="-6.0212 76.51163 16.154" rpy="1.5708 0 3.14159"/>
+      <origin xyz="0.00602 -0.07651 0.01615" rpy="0 0 0"/>
       <parent link="link_chassis"/>
       <child link="link_wheel_right"/>
-      <axis xyz="0 0 1.0"/>
+      <axis xyz="0 -1.0 0"/>
       <limit lower="-3.14" upper="3.14" effort="0" velocity="0"/>
     </joint>

Commit message: new meshes

File: description/robot.urdf.xacro (robot description, xacro)
@@ -11,5 +11,5 @@
         <origin xyz="0 0 0" rpy="0 0 0"/>
         <geometry>
-          <mesh filename="file://$(find wally)/meshes/dae/Cube.018.dae" scale="1.0 1.0 1.0"/>
+          <mesh filename="file://$(find wally)/meshes/stl/Cube.018.stl" scale="1.0 1.0 1.0"/>
         </geometry>
         <material name="black"/>
@@ -18,5 +18,5 @@
         <origin xyz="0.00012 -5e-05 6e-05" rpy="0 0 0"/>
         <geometry>
-          <mesh filename="file://$(find wally)/meshes/dae/Cube.028.dae" scale="1.0 1.0 1.0"/>
+          <mesh filename="file://$(find wally)/meshes/stl/Cube.028.stl" scale="1.0 1.0 1.0"/>
         </geometry>
       </collision>
@@ -31,5 +31,5 @@
         <origin xyz="0 0 0" rpy="0 0 0"/>
         <geometry>
-          <mesh filename="file://$(find wally)/meshes/dae/Cube.023.dae" scale="1.0 1.0 1.0"/>
+          <mesh filename="file://$(find wally)/meshes/stl/Cube.023.stl" scale="1.0 1.0 1.0"/>
         </geometry>
         <material name="yellow"/>
@@ -38,5 +38,5 @@
         <origin xyz="9e-05 0.00061 0.00011" rpy="0 0 0"/>
         <geometry>
-          <mesh filename="file://$(find wally)/meshes/dae/Cube.026.dae" scale="1.0 1.0 1.0"/>
+          <mesh filename="file://$(find wally)/meshes/stl/Cube.026.stl" scale="1.0 1.0 1.0"/>
         </geometry>
       </collision>
@@ -51,5 +51,5 @@
         <origin xyz="0 0 0" rpy="0 0 0"/>
         <geometry>
-          <mesh filename="file://$(find wally)/meshes/dae/Cube.019.dae" scale="1.0 1.0 1.0"/>
+          <mesh filename="file://$(find wally)/meshes/stl/Cube.019.stl" scale="1.0 1.0 1.0"/>
         </geometry>
         <material name="black"/>
@@ -58,5 +58,5 @@
         <origin xyz="0 0 -2e-05" rpy="0 0 0"/>
         <geometry>
-          <mesh filename="file://$(find wally)/meshes/dae/Cube.027.dae" scale="1.0 1.0 1.0"/>
+          <mesh filename="file://$(find wally)/meshes/stl/Cube.027.stl" scale="1.0 1.0 1.0"/>
         </geometry>
       </collision>
@@ -71,5 +71,5 @@
         <origin xyz="0 0 0" rpy="0 0 0"/>
         <geometry>
-          <mesh filename="file://$(find wally)/meshes/dae/Cube.020.dae" scale="1.0 1.0 1.0"/>
+          <mesh filename="file://$(find wally)/meshes/stl/Cube.020.stl" scale="1.0 1.0 1.0"/>
         </geometry>
         <material name="black"/>
@@ -85,5 +85,5 @@
         <origin xyz="0 0 0" rpy="0 0 0"/>
         <geometry>
-          <mesh filename="file://$(find wally)/meshes/dae/Cube.022.dae" scale="1.0 1.0 1.0"/>
+          <mesh filename="file://$(find wally)/meshes/stl/Cube.022.stl" scale="1.0 1.0 1.0"/>
         </geometry>
         <material name="yellow"/>
@@ -92,5 +92,5 @@
         <origin xyz="2e-05 -0.00011 2e-05" rpy="0 0 0"/>
         <geometry>
-          <mesh filename="file://$(find wally)/meshes/dae/Cube.025.dae" scale="1.0 1.0 1.0"/>
+          <mesh filename="file://$(find wally)/meshes/stl/Cube.025.stl" scale="1.0 1.0 1.0"/>
         </geometry>
       </collision>
@@ -105,5 +105,5 @@
         <origin xyz="0 0 0" rpy="0 0 0"/>
         <geometry>
-          <mesh filename="file://$(find wally)/meshes/dae/Cube.017.dae" scale="1.0 1.0 1.0"/>
+          <mesh filename="file://$(find wally)/meshes/stl/Cube.017.stl" scale="1.0 1.0 1.0"/>
         </geometry>
         <material name="yellow"/>
@@ -112,5 +112,5 @@
         <origin xyz="2e-05 0.00255 2e-05" rpy="0 0 0"/>
         <geometry>
-          <mesh filename="file://$(find wally)/meshes/dae/Cube.024.dae" scale="1.0 1.0 1.0"/>
+          <mesh filename="file://$(find wally)/meshes/stl/Cube.024.stl" scale="1.0 1.0 1.0"/>
         </geometry>
       </collision>

Commit message: new meshes and urdf

File: description/robot.urdf.xacro (robot description, xacro)
@@ -78,19 +78,19 @@
     <link name="link_wheel_left">
       <inertial>
-        <origin xyz="0 0 0" rpy="0 0 0"/>
+        <origin xyz="0 0.00527 0" rpy="0 0 0"/>
         <mass value="1.0"/>
-        <inertia ixx="289.20636" ixy="0" ixz="0" iyy="506.04105" iyz="0" izz="289.19714"/>
+        <inertia ixx="2e-05" ixy="0" ixz="0" iyy="2e-05" iyz="0" izz="2e-05"/>
       </inertial>
       <visual name="wheel_left">
-        <origin xyz="0 0 0" rpy="0 0 0"/>
+        <origin xyz="0 0.00264 0" rpy="0 0 0"/>
         <geometry>
-          <mesh filename="file://$(find wally)/meshes/stl/Cube.022.stl" scale="1.0 1.0 1.0"/>
+          <mesh filename="file://$(find wally)/meshes/stl/Cylinder.036.stl" scale="1.0 1.0 1.0"/>
         </geometry>
-        <material name="yellow"/>
+        <material name="black"/>
       </visual>
       <collision name="wheel_left">
-        <origin xyz="2e-05 -0.00011 2e-05" rpy="0 0 0"/>
+        <origin xyz="0 0 0" rpy="1.5708 0 0"/>
         <geometry>
-          <mesh filename="file://$(find wally)/meshes/stl/Cube.025.stl" scale="1.0 1.0 1.0"/>
+          <cylinder radius="0.03446" length="0.03"/>
         </geometry>
       </collision>
@@ -98,19 +98,19 @@
     <link name="link_wheel_right">
       <inertial>
-        <origin xyz="0 0 0" rpy="0 0 0"/>
+        <origin xyz="0 -0.00632 0" rpy="0 0 0"/>
         <mass value="1.0"/>
-        <inertia ixx="289.20636" ixy="0" ixz="0" iyy="506.04105" iyz="0" izz="289.19717"/>
+        <inertia ixx="2e-05" ixy="0" ixz="0" iyy="2e-05" iyz="0" izz="2e-05"/>
       </inertial>
       <visual name="wheel_right">
-        <origin xyz="0 0 0" rpy="0 0 0"/>
+        <origin xyz="0 -0.00316 0" rpy="0 0 0"/>
         <geometry>
-          <mesh filename="file://$(find wally)/meshes/stl/Cube.017.stl" scale="1.0 1.0 1.0"/>
+          <mesh filename="file://$(find wally)/meshes/stl/Cylinder.037.stl" scale="1.0 1.0 1.0"/>
         </geometry>
-        <material name="yellow"/>
+        <material name="black"/>
       </visual>
       <collision name="wheel_right">
-        <origin xyz="2e-05 0.00255 2e-05" rpy="0 0 0"/>
+        <origin xyz="0 -0.00052 0" rpy="1.5708 0 0"/>
         <geometry>
-          <mesh filename="file://$(find wally)/meshes/stl/Cube.024.stl" scale="1.0 1.0 1.0"/>
+          <cylinder radius="0.03446" length="0.03"/>
         </geometry>
       </collision>

Commit message: simulation update, getting ready for real robot

File: description/robot.urdf.xacro (robot description, xacro)
@@ -1,153 +1,15 @@
 <?xml version="1.0"?>
-<!-- created with Phobos 1.0.1 "Capricious Choutengan" -->
-  <robot name="wally">
-    <link name="link_camera">
-      <inertial>
-        <origin xyz="0 0 0" rpy="0 0 0"/>
-        <mass value="1.0"/>
-        <inertia ixx="288.5336" ixy="0" ixz="0" iyy="274.41498" iyz="0" izz="149.48827"/>
-      </inertial>
-      <visual name="camera">
-        <origin xyz="0 0 0" rpy="0 0 0"/>
-        <geometry>
-          <mesh filename="file://$(find wally)/meshes/stl/Cube.018.stl" scale="1.0 1.0 1.0"/>
-        </geometry>
-        <material name="black"/>
-      </visual>
-      <collision name="camera">
-        <origin xyz="0.00012 -5e-05 6e-05" rpy="0 0 0"/>
-        <geometry>
-          <mesh filename="file://$(find wally)/meshes/stl/Cube.028.stl" scale="1.0 1.0 1.0"/>
-        </geometry>
-      </collision>
-    </link>
-    <link name="link_chassis">
-      <inertial>
-        <origin xyz="0 0 0" rpy="0 0 0"/>
-        <mass value="1.0"/>
-        <inertia ixx="2658.80078" ixy="0" ixz="0" iyy="4901.40967" iyz="0" izz="5801.34521"/>
-      </inertial>
-      <visual name="chassis">
-        <origin xyz="0 0 0" rpy="0 0 0"/>
-        <geometry>
-          <mesh filename="file://$(find wally)/meshes/stl/Cube.023.stl" scale="1.0 1.0 1.0"/>
-        </geometry>
-        <material name="yellow"/>
-      </visual>
-      <collision name="chassis">
-        <origin xyz="9e-05 0.00061 0.00011" rpy="0 0 0"/>
-        <geometry>
-          <mesh filename="file://$(find wally)/meshes/stl/Cube.026.stl" scale="1.0 1.0 1.0"/>
-        </geometry>
-      </collision>
-    </link>
-    <link name="link_laser">
-      <inertial>
-        <origin xyz="0 0 0" rpy="0 0 0"/>
-        <mass value="1.0"/>
-        <inertia ixx="297.87347" ixy="0" ixz="0" iyy="297.87271" iyz="0" izz="224.89485"/>
-      </inertial>
-      <visual name="laser">
-        <origin xyz="0 0 0" rpy="0 0 0"/>
-        <geometry>
-          <mesh filename="file://$(find wally)/meshes/stl/Cube.019.stl" scale="1.0 1.0 1.0"/>
-        </geometry>
-        <material name="black"/>
-      </visual>
-      <collision name="laser">
-        <origin xyz="0 0 -2e-05" rpy="0 0 0"/>
-        <geometry>
-          <mesh filename="file://$(find wally)/meshes/stl/Cube.027.stl" scale="1.0 1.0 1.0"/>
-        </geometry>
-      </collision>
-    </link>
-    <link name="link_wheel_caster">
-      <inertial>
-        <origin xyz="0 0 0" rpy="0 0 0"/>
-        <mass value="1.0"/>
-        <inertia ixx="59.09788" ixy="0" ixz="0" iyy="40.71418" iyz="0" izz="77.59837"/>
-      </inertial>
-      <visual name="wheel_caster">
-        <origin xyz="0 0 0" rpy="0 0 0"/>
-        <geometry>
-          <mesh filename="file://$(find wally)/meshes/stl/Cube.020.stl" scale="1.0 1.0 1.0"/>
-        </geometry>
-        <material name="black"/>
-      </visual>
-    </link>
-    <link name="link_wheel_left">
-      <inertial>
-        <origin xyz="0 0.00527 0" rpy="0 0 0"/>
-        <mass value="1.0"/>
-        <inertia ixx="2e-05" ixy="0" ixz="0" iyy="2e-05" iyz="0" izz="2e-05"/>
-      </inertial>
-      <visual name="wheel_left">
-        <origin xyz="0 0.00264 0" rpy="0 0 0"/>
-        <geometry>
-          <mesh filename="file://$(find wally)/meshes/stl/Cylinder.036.stl" scale="1.0 1.0 1.0"/>
-        </geometry>
-        <material name="black"/>
-      </visual>
-      <collision name="wheel_left">
-        <origin xyz="0 0 0" rpy="1.5708 0 0"/>
-        <geometry>
-          <cylinder radius="0.03446" length="0.03"/>
-        </geometry>
-      </collision>
-    </link>
-    <link name="link_wheel_right">
-      <inertial>
-        <origin xyz="0 -0.00632 0" rpy="0 0 0"/>
-        <mass value="1.0"/>
-        <inertia ixx="2e-05" ixy="0" ixz="0" iyy="2e-05" iyz="0" izz="2e-05"/>
-      </inertial>
-      <visual name="wheel_right">
-        <origin xyz="0 -0.00316 0" rpy="0 0 0"/>
-        <geometry>
-          <mesh filename="file://$(find wally)/meshes/stl/Cylinder.037.stl" scale="1.0 1.0 1.0"/>
-        </geometry>
-        <material name="black"/>
-      </visual>
-      <collision name="wheel_right">
-        <origin xyz="0 -0.00052 0" rpy="1.5708 0 0"/>
-        <geometry>
-          <cylinder radius="0.03446" length="0.03"/>
-        </geometry>
-      </collision>
-    </link>
-    <joint name="link_camera" type="fixed">
-      <origin xyz="0.0995 0.00066 0.07561" rpy="0 0 0"/>
-      <parent link="link_chassis"/>
-      <child link="link_camera"/>
-    </joint>
-    <joint name="link_laser" type="fixed">
-      <origin xyz="-0.01313 0.00061 0.1045" rpy="0 0 0"/>
-      <parent link="link_chassis"/>
-      <child link="link_laser"/>
-    </joint>
-    <joint name="link_wheel_caster" type="fixed">
-      <origin xyz="-0.09896 0.00061 -0.00789" rpy="0 0 0"/>
-      <parent link="link_chassis"/>
-      <child link="link_wheel_caster"/>
-    </joint>
-    <joint name="link_wheel_left" type="revolute">
-      <origin xyz="0.00602 0.07703 0.01615" rpy="0 0 0"/>
-      <parent link="link_chassis"/>
-      <child link="link_wheel_left"/>
-      <axis xyz="0 1.0 0"/>
-      <limit lower="-3.14" upper="3.14" effort="0" velocity="0"/>
-    </joint>
-    <joint name="link_wheel_right" type="revolute">
-      <origin xyz="0.00602 -0.07651 0.01615" rpy="0 0 0"/>
-      <parent link="link_chassis"/>
-      <child link="link_wheel_right"/>
-      <axis xyz="0 -1.0 0"/>
-      <limit lower="-3.14" upper="3.14" effort="0" velocity="0"/>
-    </joint>
-    <material name="black">
-      <color rgba="0.8 0.8 0.8 1.0"/>
-    </material>
-    <material name="yellow">
-      <color rgba="0.8 0.8 0.8 1.0"/>
-    </material>
-  </robot>
+<robot xmlns:xacro="http://www.ros.org/wiki/xacro"  name="robot">
+    <xacro:arg name="use_ros2_control" default="true"/>
+    <xacro:include filename="robot_core_2.xacro"/>
+    <xacro:include filename="lidar.xacro"/>
+    <xacro:include filename="camera.xacro"/>
+    <!--<xacro:include filename="gazebo_control.xacro"/>-->
+    <xacro:if value="$(arg use_ros2_control)">
+        <xacro:include filename="ros2_control.xacro" />
+    </xacro:if>
+    <xacro:unless value="$(arg use_ros2_control)">
+        <xacro:include filename="gazebo_control.xacro" />
+    </xacro:unless>
+    <!--<xacro:include filename="ros2_control.xacro" />-->
+</robot>
