Commit message: More non-sim changes

File: description/robot.urdf.xacro (robot description, xacro)
@@ -2,8 +2,5 @@
 <robot xmlns:xacro="http://www.ros.org/wiki/xacro"  name="robot">
     <xacro:arg name="use_ros2_control" default="true"/>
-    <xacro:include filename="robot_core_2.xacro"/>
-    <xacro:include filename="lidar.xacro"/>
-    <xacro:include filename="camera.xacro"/>
-    <!--<xacro:include filename="gazebo_control.xacro"/>-->
+    <xacro:include filename="robot_core_2.xacro" />
     <xacro:if value="$(arg use_ros2_control)">
         <xacro:include filename="ros2_control.xacro" />
@@ -12,4 +9,5 @@
         <xacro:include filename="gazebo_control.xacro" />
     </xacro:unless>
-    <!--<xacro:include filename="ros2_control.xacro" />-->
+    <xacro:include filename="lidar.xacro" />
+    <xacro:include filename="camera.xacro" />
 </robot>

File: description/robot_core_2.xacro (robot description, xacro)
@@ -9,11 +9,12 @@
     <xacro:property name="wheel_thickness" value="0.026" />
     <xacro:property name="wheel_mass" value="0.5" />
-    <xacro:property name="wheel_offset_x" value="0.015" />
+    <xacro:property name="wheel_offset_x" value="0.025" />
     <xacro:property name="wheel_offset_y" value="${chassis_width/2 + wheel_thickness/2 - 0.01}" />
-    <xacro:property name="wheel_offset_z" value="0.014" />
+    <xacro:property name="wheel_offset_z" value="-${chassis_width/2 - 0.036}" />
     <xacro:property name="caster_wheel_radius" value="0.012" />
     <xacro:property name="caster_wheel_mass" value="0.5" />
     <xacro:property name="caster_wheel_offset_x" value="-0.08" />
     <xacro:property name="caster_wheel_offset_z" value="-0.058" />
+    <xacro:property name="meshpath" value="/home/dev/dev_ws/src/wally" />
     <material name="yellow">
         <color rgba="1 1 0 1 " />
@@ -46,5 +47,5 @@
         <visual>
             <geometry>
-                <mesh filename="file://$(find wally)/meshes/stl/Cube.023.stl" scale="1.0 1.0 1.0"/>
+                <mesh filename="file://${meshpath}/meshes/stl/Cube.023.stl" scale="1.0 1.0 1.0"/>
                 <!--<box size="${chassis_length} ${chassis_width} ${chassis_height}"/>-->
             </geometry>
@@ -67,5 +68,5 @@
     <joint name="left_wheel_joint" type="continuous">
         <origin xyz="${wheel_offset_x} ${wheel_offset_y} ${wheel_offset_z}" rpy="-${pi/2} 0 0"/>
-        <parent link="base_link"/>
+        <parent link="chassis"/>
         <child link="left_wheel"/>
         <axis xyz="0 0 1"/>
@@ -75,5 +76,5 @@
             <geometry>
                 <!--<cylinder radius="${wheel_radius}" length="${wheel_thickness}"/>-->
-                <mesh filename="file://$(find wally)/meshes/stl/Cylinder.036.stl" scale="1.0 1.0 1.0"/>
+                <mesh filename="file://${meshpath}/meshes/stl/Cylinder.036.stl" scale="1.0 1.0 1.0"/>
             </geometry>
             <material name="yellow"/>
@@ -94,5 +95,5 @@
     <joint name="right_wheel_joint" type="continuous">
         <origin xyz="${wheel_offset_x} -${wheel_offset_y} ${wheel_offset_z}" rpy="${pi/2} 0 0"/>
-        <parent link="base_link"/>
+        <parent link="chassis"/>
         <child link="right_wheel"/>
         <axis xyz="0 0 -1"/>
@@ -102,5 +103,5 @@
             <geometry>
                 <!--<cylinder radius="${wheel_radius}" length="${wheel_thickness}"/>-->
-                <mesh filename="file://$(find wally)/meshes/stl/Cylinder.036.stl" scale="1.0 1.0 1.0"/>
+                <mesh filename="file://${meshpath}/meshes/stl/Cylinder.036.stl" scale="1.0 1.0 1.0"/>
             </geometry>
             <material name="yellow"/>
@@ -128,5 +129,5 @@
             <geometry>
                 <!--<sphere radius="${caster_wheel_radius}"/>-->
-                <mesh filename="file://$(find wally)/meshes/stl/Cube.020.stl" scale="1.0 1.0 1.0"/>
+                <mesh filename="file://${meshpath}/meshes/stl/Cube.020.stl" scale="1.0 1.0 1.0"/>
             </geometry>
             <material name="grey"/>

File: description/ros2_control.xacro (robot description, xacro)
@@ -1,7 +1,14 @@
 <?xml version="1.0"?>
 <robot xmlns:xacro="http://www.ros.org/wiki/xacro">
-        <ros2_control name="GazeboSystem" type="system">
+        <ros2_control name="RealRobot" type="system">
             <hardware>
-                <plugin>gazebo_ros2_control/GazeboSystem</plugin>
+                <plugin>diffdrive_arduino/DiffDriveArduino</plugin>
+                <param name="left_wheel_name">left_wheel_joint</param>
+                <param name="right_wheel_name">right_wheel_joint</param>
+                <param name="loop_rate">30</param>
+                <param name="device">/dev/ttyUSB0</param>
+                <param name="baud_rate">57600</param>
+                <param name="timeout">1000</param>
+                <param name="enc_counts_per_rev">3880</param>
             </hardware>
             <joint name="left_wheel_joint">
@@ -22,4 +29,25 @@
             </joint>
         </ros2_control>
+    <!-- <ros2_control name="GazeboSystem" type="system">
+        <hardware>
+            <plugin>gazebo_ros2_control/GazeboSystem</plugin>
+        </hardware>
+        <joint name="left_wheel_joint">
+            <command_interface name="velocity">
+                <param name="min">-10</param>
+                <param name="max">10</param>
+            </command_interface>
+            <state_interface name="velocity"/>
+            <state_interface name="position"/>
+        </joint>
+        <joint name="right_wheel_joint">
+            <command_interface name="velocity">
+                <param name="min">-10</param>
+                <param name="max">10</param>
+            </command_interface>
+            <state_interface name="velocity"/>
+            <state_interface name="position"/>
+        </joint>
+    </ros2_control> -->
     <gazebo>
         <plugin name="gazebo_ros2_control" filename="libgazebo_ros2_control.so">
